Commit message: rplidar urdf

File: icerobot/icerobot_description/urdf/lidar.urdf.xacro (robot description, xacro)
@@ -68,5 +68,5 @@
       <parent link="${parent_link}"/>
       <child link="rplidar_scan"/>
-      <origin xyz="0.3 0.007 0.615" rpy="0 0 0"/>
+      <origin xyz="0.29 0.075 0.615" rpy="0 0 ${PI}"/>
     </joint>
     <link name="rplidar_scan">
