Commit message: localization fixtures

File: icerobot/icerobot_description/urdf/imu.urdf.xacro (robot description, xacro)
@@ -5,5 +5,5 @@
     <link name="um7_imu_link"/>
     <joint name="um7_imu_joint" type="fixed">
-      <origin xyz="-0.10 0.007 1.28" rpy="0 0 0" />
+	    <origin xyz="-0.10 0.007 1.28" rpy="${PI} 0 0" />
       <parent link="${parent_link}" />
       <child link="um7_imu_link" />

Commit message: fix merges

File: icerobot/icerobot_description/urdf/imu.urdf.xacro (robot description, xacro)
@@ -5,5 +5,5 @@
     <link name="um7_imu_link"/>
     <joint name="um7_imu_joint" type="fixed">
-	    <origin xyz="-0.10 0.007 1.28" rpy="${PI} 0 0" />
+	    <origin xyz="-0.10 0.007 1.28" rpy="0 0 0" />
       <parent link="${parent_link}" />
       <child link="um7_imu_link" />
