Commit message: drive & lidar fix

File: icerobot/icerobot_description/urdf/icerobot.urdf.xacro (robot description, xacro)
@@ -168,5 +168,5 @@
     <parent link="base_link"/>
     <child link="base_scan"/>
-    <origin xyz="-0.375 0.008 1.322" rpy="${PI/2} 0 ${PI/2+PI}"/>
+    <origin xyz="-0.375 0.008 1.322" rpy="0 ${-PI/2} 0"/>
   </joint>
   <link name="base_scan">

Commit message: gazebo fix

File: icerobot/icerobot_description/urdf/icerobot.urdf.xacro (robot description, xacro)
@@ -8,8 +8,8 @@
   <xacro:property name="base_x_size" value="0.96520000" />
   <xacro:property name="base_y_size" value="0.63500000" />
-  <xacro:property name="base_z_size" value="0.6154100" />
+  <xacro:property name="base_z_size" value="0.5754100" />
   <!-- Platform Size -->
-  <xacro:property name="platform_x_size" value="0.320000" />
-  <xacro:property name="platform_y_size" value="0.63500000" />
+  <xacro:property name="platform_x_size" value="0.100000" />
+  <xacro:property name="platform_y_size" value="0.100000" />
   <xacro:property name="platform_z_size" value="1.4000000" />
   <!-- Wheel Mounting Positions -->
@@ -90,5 +90,5 @@
         <box size="${platform_x_size} ${platform_y_size} ${platform_z_size}"/>
       </geometry>
-      <origin rpy="0 0 0" xyz="0.1 0 ${(platform_z_size/2)}"/>
+      <origin rpy="0 0 0" xyz="0.18 0 ${(platform_z_size/2)}"/>
     </collision>
     <inertial>

File: icerobot/icerobot_description/urdf/imu.urdf.xacro (robot description, xacro)
@@ -15,5 +15,5 @@
         <robotNamespace>$(arg robot_namespace)</robotNamespace>
         <updateRate>20.0</updateRate>
-        <bodyName>um7_imu_link</bodyName>
+        <bodyName>${parent_link}</bodyName>
         <topicName>${topic_imu_um7}</topicName>
         <xyzOffset>0 0 0</xyzOffset>
@@ -40,5 +40,5 @@
         <robotNamespace>$(arg robot_namespace)</robotNamespace>
         <updateRate>20.0</updateRate>
-        <bodyName>azure_imu_link</bodyName>
+	<bodyName>${parent_link}</bodyName>
         <topicName>${topic_imu_azure}</topicName>
         <xyzOffset>0 0 0</xyzOffset>

File: icerobot/icerobot_description/urdf/lidar.urdf.xacro (robot description, xacro)
@@ -23,5 +23,5 @@
       </inertial>
     </link>
-    <gazebo reference="vlp16_base_scan">
+    <gazebo reference="vlp16_scan">
       <sensor type="ray" name="velodyne_VLP16">
         <pose>2 0 0 0 0 0</pose>
@@ -56,6 +56,6 @@
         <plugin name="gazebo_ros_laser_controller" filename="libgazebo_ros_laser.so">
           <robotNamespace>$(arg robot_namespace)</robotNamespace>
-          <topicName>${topic_lidar_vlp16}</topicName>
-          <frameName>vlp16_base_scan</frameName>
+	  <topicName>${topic_lidar_vlp16}</topicName>
+          <frameName>vlp16_scan</frameName>
           <min_range>0.9</min_range>
           <max_range>130</max_range>
@@ -68,9 +68,9 @@
       <parent link="${parent_link}"/>
       <child link="rplidar_scan"/>
-      <origin xyz="0.3 0.007 0.6" rpy="0 0 0"/>
+      <origin xyz="0.3 0.007 0.615" rpy="0 0 0"/>
     </joint>
     <link name="rplidar_scan">
       <visual>
-        <origin xyz="0 0 0" rpy="0 0 0"/>
+        <origin xyz="0 0 -0.025" rpy="0 0 0"/>
         <geometry>
           <mesh filename="package://icerobot_description/meshes/rplidar.dae"/>
@@ -86,6 +86,6 @@
     </link>
   <!-- RpLidar A3 using GPU -->
-    <gazebo reference="rplidar_base_scan">
-      <sensor type="gpu_ray" name="head_rplidar_sensor">
+    <gazebo reference="rplidar_scan">
+      <sensor type="ray" name="head_rplidar_sensor">
         <pose>0 0 0.06 0 0 0</pose>
         <visualize>false</visualize>
@@ -111,7 +111,7 @@
           </noise>
         </ray>
-        <plugin name="gazebo_ros_head_rplidar_controller" filename="libgazebo_ros_gpu_laser.so">
+        <plugin name="gazebo_ros_head_rplidar_controller" filename="libgazebo_ros_laser.so">
           <topicName>${topic_lidar_rplidar}</topicName>
-          <frameName>rplidar_base_scan</frameName>
+          <frameName>rplidar_scan</frameName>
         </plugin>
       </sensor>

File: icerobot/icerobot_description/urdf/wheels.urdf.xacro (robot description, xacro)
@@ -31,6 +31,6 @@
     <!-- Wheel parameters -->
     <gazebo reference="${prefix}_${suffix}_wheel">
-      <mu1 value="0.09"/>
-      <mu2 value="0.35"/>
+      <mu1 value="0.35"/>
+      <mu2 value="0.09"/>
       <kp value="100000000.0" />
       <kd value="1.0" />

Commit message: gps urdf add

File: icerobot/icerobot_description/urdf/icerobot.urdf.xacro (robot description, xacro)
@@ -108,4 +108,10 @@
     <child link="base_footprint" />
   </joint>
+  <link name="gps_link"/>
+  <joint name="gps_joint" type="fixed">
+    <origin xyz="0.05 0.007 1.75" rpy="0 0 0" />
+    <parent link="base_link" />
+    <child link="gps_link" />
+  </joint>
   <!-- Wheel xacro -->
   <xacro:wheel prefix="front" suffix="left" reflect_side="1" reflect_front="1"/>

Commit message: gazebo & localization fix

File: icerobot/icerobot_description/urdf/icerobot.urdf.xacro (robot description, xacro)
@@ -21,27 +21,27 @@
   <xacro:property name="wheel_radius" value="0.167" />
   <!-- Base inertia properties -->
-  <xacro:property name="mass_base" value="34.33" />
-  <xacro:property name="ixx_base" value="2.4304" />
-  <xacro:property name="ixy_base" value="0.5116" />
-  <xacro:property name="ixz_base" value="0.0091" />
-  <xacro:property name="iyy_base" value="3.7564" />
-  <xacro:property name="iyz_base" value="-0.0016" />
-  <xacro:property name="izz_base" value="3.8077" />
+  <xacro:property name="mass_base" value="49.7354" />
+  <xacro:property name="ixx_base" value="2.6820" />
+  <xacro:property name="ixy_base" value="0.5001" />
+  <xacro:property name="ixz_base" value="0.0135" />
+  <xacro:property name="iyy_base" value="4.3224" />
+  <xacro:property name="iyz_base" value="-0.0044" />
+  <xacro:property name="izz_base" value="4.3573" />
   <!-- Platform inertia properties -->
-  <xacro:property name="mass_platform" value="49.4938" />
-  <xacro:property name="ixx_platform" value="16.83" />
-  <xacro:property name="ixy_platform" value="0.3363" />
-  <xacro:property name="ixz_platform" value="0.1616" />
-  <xacro:property name="iyy_platform" value="3.9954" />
-  <xacro:property name="iyz_platform" value="6.3377" />
-  <xacro:property name="izz_platform" value="13.2782" />
+  <xacro:property name="mass_platform" value="10.9227" />
+  <xacro:property name="ixx_platform" value="7.8672" />
+  <xacro:property name="ixy_platform" value="0.5195" />
+  <xacro:property name="ixz_platform" value="0.0006" />
+  <xacro:property name="iyy_platform" value="0.3726" />
+  <xacro:property name="iyz_platform" value="0.0069" />
+  <xacro:property name="izz_platform" value="8.1169" />
   <!-- Wheel inertia properties -->
-  <xacro:property name="mass_wheel" value="4" />
-  <xacro:property name="ixx_wheel" value="0.0553" />
-  <xacro:property name="ixy_wheel" value="0" />
-  <xacro:property name="ixz_wheel" value="0" />
-  <xacro:property name="iyy_wheel" value="0.0315" />
-  <xacro:property name="iyz_wheel" value="0" />
-  <xacro:property name="izz_wheel" value="0.0315" />
+  <xacro:property name="mass_wheel" value="4.3340" />
+  <xacro:property name="ixx_wheel" value="0.6036" />
+  <xacro:property name="ixy_wheel" value="0.1952" />
+  <xacro:property name="ixz_wheel" value="0.4462" />
+  <xacro:property name="iyy_wheel" value="0.9226" />
+  <xacro:property name="iyz_wheel" value="0.2116" />
+  <xacro:property name="izz_wheel" value="0.5513" />
   <xacro:arg name="robot_namespace" default="/" />
   <xacro:property name="PI" value="3.14159"/>
@@ -132,5 +132,5 @@
     <plugin name="gps_controller" filename="libhector_gazebo_ros_gps.so">
       <robotNamespace>$(arg robot_namespace)</robotNamespace>
-      <updateRate>40</updateRate>
+      <updateRate>10</updateRate>
       <bodyName>base_link</bodyName>
       <frameId>base_link</frameId>

File: icerobot/icerobot_description/urdf/imu.urdf.xacro (robot description, xacro)
@@ -9,5 +9,11 @@
       <child link="um7_imu_link" />
     </joint>
-    <gazebo reference="um7_imu_link">
+    <link name="um7_imu_link_gazebo"/>
+    <joint name="um7_imu_joint_gazebo" type="fixed">
+      <origin xyz="0 0 0" rpy="0 0 0" />
+      <parent link="um7_imu_link" />
+      <child link="um7_imu_link_gazebo" />
+    </joint>
+    <gazebo reference="um7_imu_link_gazebo">
     </gazebo>
     <gazebo>
@@ -18,5 +24,5 @@
         <topicName>${topic_imu_um7}</topicName>
         <xyzOffset>0 0 0</xyzOffset>
-        <rpyOffset>0 0 0</rpyOffset>
+        <rpyOffset>0 0 1.57</rpyOffset>
         <accelDrift>0 0 0</accelDrift>
         <accelGaussianNoise>0 0 0</accelGaussianNoise>
