Commit message: sensor fix

File: icerobot/icerobot_description/urdf/azure_camera.urdf.xacro (robot description, xacro)
@@ -2,4 +2,86 @@
 <robot xmlns:xacro="http://ros.org/wiki/xacro">
   <xacro:macro name="rgbd_cameras" params="topic_azure topic_kinect parent_link">
+    <!-- Azure camera joints -->
+    <joint name="azure_camera_base_joint" type="fixed">
+      <origin xyz="-0.10 0.007 1.345" rpy="0 0 -${PI/2}"/>
+      <parent link="${parent_link}"/>
+      <child link="azure_camera_body"/>
+    </joint>
+    <link name="azure_camera_body">
+      <visual>
+        <origin xyz="0 0 0" rpy="0 0 0"/>
+        <geometry>
+         <mesh filename="package://icerobot_description/meshes/camera.dae" />
+        </geometry>
+      </visual>
+      <collision>
+        <origin xyz="0 0 0" rpy="0 0 0"/>
+        <geometry>
+          <box size="0.012 0.132 0.020"/>
+        </geometry>
+      </collision>
+      <inertial>
+        <mass value="0.44" />
+        <origin xyz="0 0 0" />
+        <inertia ixx="0.000881243" ixy="0.0" ixz="0.0"
+                 iyy="0.000498940" iyz="0.0"
+                 izz="0.000879257" />
+      </inertial>
+    </link>
+    <joint name="azure_camera_visor_joint" type="fixed">
+      <origin xyz="0.1 0 0" rpy="0 0 0"/>
+      <parent link="azure_camera_body"/>
+      <child link="azure_camera_visor"/>
+    </joint>
+    <link name="azure_camera_visor"/>
+    <joint name="azure_rgb_camera_joint" type="fixed">
+      <origin xyz="0 0 0" rpy="0 0 0"/>
+      <parent link="azure_camera_visor"/>
+      <child link="azure_rgb_camera_link"/>
+    </joint>
+    <link name="azure_rgb_camera_link"/>
+    <joint name="azure_imu_joint" type="fixed">
+      <origin xyz="0 0 0" rpy="0 0 ${PI/2}"/>
+      <parent link="azure_camera_body"/>
+      <child link="azure_imu_link"/>
+    </joint>
+    <link name="azure_imu_link"/>
+    <joint name="azure_lens_gazebo_joint" type="fixed">
+	    <origin xyz="0 0 0" rpy="0 0 0"/>
+      <parent link="azure_camera_visor"/>
+      <child link="azure_camera"/>
+    </joint>
+    <!-- Kinect camera joints -->
+    <joint name="kinect_camera_joint" type="fixed">
+      <origin xyz="0.3 0.007 0.65" rpy="0 0 0"/>
+      <parent link="${parent_link}"/>
+      <child link="kinect_camera_link"/>
+    </joint>
+    <link name="kinect_camera_link">
+      <collision>
+        <origin xyz="0 0 0" rpy="0 0 0"/>
+        <geometry>
+          <box size="0.012 0.132 0.020"/>
+        </geometry>
+      </collision>
+      <inertial>
+        <mass value="0.44" />
+        <origin xyz="0 0 0" />
+        <inertia ixx="0.000881243" ixy="0.0" ixz="0.0"
+                 iyy="0.000498940" iyz="0.0"
+                 izz="0.000879257" />
+      </inertial>
+    </link>
+    <joint name="kinect_lens_joint" type="fixed">
+      <origin xyz="0.1 0 0" rpy="0 0 0"/>
+      <parent link="kinect_camera_link"/>
+      <child link="kinect_lens_frame"/>
+    </joint>
+    <link name="kinect_lens_frame"/>
+    <joint name="kinect_lens_gazebo_joint" type="fixed">
+      <origin xyz="0 0 0" rpy="0 0 0"/>
+      <parent link="kinect_lens_frame"/>
+      <child link="kinect_camera"/>
+    </joint>
     <xacro:macro name="depth_cam_init" params="
                frame:=cam_name           topic:=cam_topic
@@ -59,75 +141,5 @@
       </gazebo>
     </xacro:macro>
-    <!-- Azure camera joints -->
-    <joint name="azure_camera_joint" type="fixed">
-      <origin xyz="-0.10 0.007 1.345" rpy="0 0 -${PI/2}"/>
-      <parent link="${parent_link}"/>
-      <child link="azure_camera_link"/>
-    </joint>
-    <link name="azure_camera_link">
-      <visual>
-        <origin xyz="0 0 0" rpy="0 0 0"/>
-        <geometry>
-         <mesh filename="package://icerobot_description/meshes/camera.dae" />
-        </geometry>
-      </visual>
-      <collision>
-        <origin xyz="0 0 0" rpy="0 0 0"/>
-        <geometry>
-          <box size="0.012 0.132 0.020"/>
-        </geometry>
-      </collision>
-      <inertial>
-        <mass value="0.44" />
-        <origin xyz="0 0 0" />
-        <inertia ixx="0.000881243" ixy="0.0" ixz="0.0"
-                 iyy="0.000498940" iyz="0.0"
-                 izz="0.000879257" />
-      </inertial>
-    </link>
-    <joint name="azure_lens_joint" type="fixed">
-      <origin xyz="0.1 0 0" rpy="0 0 0"/>
-      <parent link="azure_camera_link"/>
-      <child link="azure_lens_frame"/>
-    </joint>
-    <link name="azure_lens_frame"/>
-    <joint name="azure_lens_gazebo_joint" type="fixed">
-      <origin xyz="0 0 0" rpy="0 0 0"/>
-      <parent link="azure_lens_frame"/>
-      <child link="azure_camera"/>
-    </joint>
     <xacro:depth_cam_init frame="azure_camera" topic="${topic_azure}"/>
-    <!-- Kinect camera joints -->
-    <joint name="kinect_camera_joint" type="fixed">
-      <origin xyz="0.3 0.007 0.65" rpy="0 0 0"/>
-      <parent link="${parent_link}"/>
-      <child link="kinect_camera_link"/>
-    </joint>
-    <link name="kinect_camera_link">
-      <collision>
-        <origin xyz="0 0 0" rpy="0 0 0"/>
-        <geometry>
-          <box size="0.012 0.132 0.020"/>
-        </geometry>
-      </collision>
-      <inertial>
-        <mass value="0.44" />
-        <origin xyz="0 0 0" />
-        <inertia ixx="0.000881243" ixy="0.0" ixz="0.0"
-                 iyy="0.000498940" iyz="0.0"
-                 izz="0.000879257" />
-      </inertial>
-    </link>
-    <joint name="kinect_lens_joint" type="fixed">
-      <origin xyz="0.1 0 0" rpy="0 0 0"/>
-      <parent link="kinect_camera_link"/>
-      <child link="kinect_lens_frame"/>
-    </joint>
-    <link name="kinect_lens_frame"/>
-    <joint name="kinect_lens_gazebo_joint" type="fixed">
-      <origin xyz="0 0 0" rpy="0 0 0"/>
-      <parent link="kinect_lens_frame"/>
-      <child link="kinect_camera"/>
-    </joint>
     <xacro:depth_cam_init frame="kinect_camera" topic="${topic_kinect}"
                           h_fov="0.9948"         v_fov="0.7505"

Commit message: fix azure tf

File: icerobot/icerobot_description/urdf/azure_camera.urdf.xacro (robot description, xacro)
@@ -4,5 +4,5 @@
     <!-- Azure camera joints -->
     <joint name="azure_camera_base_joint" type="fixed">
-      <origin xyz="-0.10 0.007 1.345" rpy="0 0 -${PI/2}"/>
+      <origin xyz="-0.10 0.007 1.345" rpy="0 0 ${-PI/2}"/>
       <parent link="${parent_link}"/>
       <child link="azure_camera_body"/>
@@ -30,15 +30,9 @@
     </link>
     <joint name="azure_camera_visor_joint" type="fixed">
-      <origin xyz="0.1 0 0" rpy="0 0 0"/>
+      <origin xyz="0.1 0 0" rpy="${-PI/2-0.2} 0 ${-PI/2}"/>
       <parent link="azure_camera_body"/>
       <child link="azure_camera_visor"/>
     </joint>
     <link name="azure_camera_visor"/>
-    <joint name="azure_rgb_camera_joint" type="fixed">
-      <origin xyz="0 0 0" rpy="0 0 0"/>
-      <parent link="azure_camera_visor"/>
-      <child link="azure_rgb_camera_link"/>
-    </joint>
-    <link name="azure_rgb_camera_link"/>
     <joint name="azure_imu_joint" type="fixed">
       <origin xyz="0 0 0" rpy="0 0 ${PI/2}"/>

Commit message: urdf update

File: icerobot/icerobot_description/urdf/azure_camera.urdf.xacro (robot description, xacro)
@@ -1,5 +1,6 @@
 <?xml version="1.0"?>
 <robot xmlns:xacro="http://ros.org/wiki/xacro">
-  <xacro:macro name="rgbd_cameras" params="topic_azure topic_kinect parent_link">
+<!-- add topic_kinect to param for kinect camera -->
+  <xacro:macro name="rgbd_cameras" params="topic_azure parent_link">
     <!-- Azure camera joints -->
     <joint name="azure_camera_base_joint" type="fixed">
@@ -10,5 +11,5 @@
     <link name="azure_camera_body">
       <visual>
-        <origin xyz="0 0 0" rpy="0 0 0"/>
+        <origin xyz="0 0 0" rpy="0 0 ${PI}"/>
         <geometry>
          <mesh filename="package://icerobot_description/meshes/camera.dae" />
@@ -30,9 +31,10 @@
     </link>
     <joint name="azure_camera_visor_joint" type="fixed">
-      <origin xyz="0.1 0 0" rpy="${-PI/2-0.2} 0 ${-PI/2}"/>
+      <origin xyz="0.07 0 0.025" rpy="${-PI/2-0.1} 0 ${-PI/2}"/>
       <parent link="azure_camera_body"/>
       <child link="azure_camera_visor"/>
     </joint>
     <link name="azure_camera_visor"/>
+<!--
     <joint name="azure_imu_joint" type="fixed">
       <origin xyz="0 0 0" rpy="0 0 ${PI/2}"/>
@@ -41,4 +43,5 @@
     </joint>
     <link name="azure_imu_link"/>
+ -->
     <joint name="azure_lens_gazebo_joint" type="fixed">
 	    <origin xyz="0 0 0" rpy="0 0 0"/>
@@ -46,5 +49,5 @@
       <child link="azure_camera"/>
     </joint>
-    <!-- Kinect camera joints -->
+    <!-- Kinect camera joints
     <joint name="kinect_camera_joint" type="fixed">
       <origin xyz="0.3 0.007 0.65" rpy="0 0 0"/>
@@ -78,4 +81,5 @@
       <child link="kinect_camera"/>
     </joint>
+    -->
     <xacro:macro name="depth_cam_init" params="
                frame:=cam_name           topic:=cam_topic
@@ -104,5 +108,4 @@
             <clip>
               <near>0.01</near>
-              <!-- Max distance -->
               <far>50.0</far>
             </clip>
@@ -136,9 +139,10 @@
     </xacro:macro>
     <xacro:depth_cam_init frame="azure_camera" topic="${topic_azure}"/>
-    <xacro:depth_cam_init frame="kinect_camera" topic="${topic_kinect}"
+    <!--<xacro:depth_cam_init frame="kinect_camera" topic="${topic_kinect}"
                           h_fov="0.9948"         v_fov="0.7505"
                           min_range="1.2"        max_range="3.5"
                           width="640"            height="480"
                           update_rate="30"/>
+    -->
   </xacro:macro>
 </robot>

File: icerobot/icerobot_description/urdf/icerobot.urdf.xacro (robot description, xacro)
@@ -2,4 +2,7 @@
 <robot name="icerobot" xmlns:xacro="http://ros.org/wiki/xacro">
   <xacro:include filename="$(find icerobot_description)/urdf/azure_camera.urdf.xacro" />
+  <xacro:include filename="$(find icerobot_description)/urdf/wheels.urdf.xacro" />
+  <xacro:include filename="$(find icerobot_description)/urdf/imu.urdf.xacro" />
+  <xacro:include filename="$(find icerobot_description)/urdf/lidar.urdf.xacro" />
   <!-- Base Size -->
   <xacro:property name="base_x_size" value="0.96520000" />
@@ -70,54 +73,4 @@
     <child link="inertial_link" />
   </joint>
-  <!-- Wheel macros -->
-  <xacro:macro name="wheel" params="prefix suffix reflect_side reflect_front">
-    <link name="${prefix}_${suffix}_wheel">
-      <visual>
-       <origin xyz="0 0 0" rpy="0 0 ${reflect_side*PI/2+PI}" />
-       <geometry>
-         <mesh filename="package://icerobot_description/meshes/wheel.dae"/>
-       </geometry>
-      </visual>
-      <collision>
-	      <origin xyz="0 ${reflect_side*0.04} 0" rpy="${PI/2} 0 0" />
-        <geometry>
-          <cylinder radius="${wheel_radius}" length="${wheel_length}"/>
-        </geometry>
-      </collision>
-      <inertial>
-        <mass value="${mass_wheel}" />
-        <origin xyz="0 0 0" />
-        <inertia ixx="${ixx_wheel}" ixy="${ixy_wheel}" ixz="${ixz_wheel}" iyy="${iyy_wheel}" iyz="${iyz_wheel}" izz="${izz_wheel}"/>
-      </inertial>
-    </link>
-    <joint name="${prefix}_${suffix}_wheel_joint" type="continuous">
-      <axis xyz="0 1 0" rpy="0 0 0" />
-      <parent link="base_link"/>
-      <child link="${prefix}_${suffix}_wheel"/>
-      <origin xyz="${reflect_front*wheelbase} ${reflect_side*track} ${wheel_vertical_offset}" rpy="0 0 0"/>
-    </joint>
-    <!-- Gazebo xacro -->
-    <!-- Wheel parameters -->
-    <gazebo reference="${prefix}_${suffix}_wheel">
-      <mu1 value="1.0"/>
-      <mu2 value="0.5"/>
-      <kp value="100000000.0" />
-      <kd value="1.0" />
-      <fdir1 value="1 0 0"/>
-    </gazebo>
-    <transmission name="${prefix}_${suffix}_wheel_trans" type="SimpleTransmission">
-      <type>transmission_interface/SimpleTransmission</type>
-      <actuator name="${prefix}_${suffix}_wheel_motor">
-        <mechanicalReduction>1</mechanicalReduction>
-      </actuator>
-      <joint name="${prefix}_${suffix}_wheel_joint">
-        <hardwareInterface>hardware_interface/VelocityJointInterface</hardwareInterface>
-      </joint>
-    </transmission>
-  </xacro:macro>
-  <xacro:wheel prefix="front" suffix="left" reflect_side="1" reflect_front="1"/>
-  <xacro:wheel prefix="rear" suffix="left" reflect_side="1" reflect_front="-1"/>
-  <xacro:wheel prefix="front" suffix="right" reflect_side="-1" reflect_front="1"/>
-  <xacro:wheel prefix="rear" suffix="right" reflect_side="-1" reflect_front="-1"/>
   <!-- Sensor Platform -->
   <joint name="platform_to_base" type="fixed">
@@ -137,5 +90,5 @@
         <box size="${platform_x_size} ${platform_y_size} ${platform_z_size}"/>
       </geometry>
-      <origin rpy="0 0 0" xyz="-0.1 0 ${(platform_z_size/2)}"/>
+      <origin rpy="0 0 0" xyz="0.1 0 ${(platform_z_size/2)}"/>
     </collision>
     <inertial>
@@ -155,61 +108,17 @@
     <child link="base_footprint" />
   </joint>
-  <!-- IMU Link is the standard mounting position for the UM6 IMU.-->
-  <!-- Can be modified with environment variables in /etc/ros/setup.bash -->
-  <link name="imu_link"/>
-  <joint name="imu_joint" type="fixed">
-	  <origin xyz="-0.10 0.007 1.24" rpy="0 0 0" />
-    <parent link="base_link" />
-    <child link="imu_link" />
-  </joint>
-  <gazebo reference="imu_link">
-  </gazebo>
-  <joint name="scan_joint" type="fixed">
-    <parent link="base_link"/>
-    <child link="base_scan"/>
-    <origin xyz="-0.375 0.008 1.322" rpy="0 ${-PI/2} 0"/>
-  </joint>
-  <link name="base_scan">
-    <visual>
-      <origin xyz="0 0 -0.1" rpy="0 0 0"/>
-      <geometry>
-        <mesh filename="package://icerobot_description/meshes/lidar.dae"/>
-      </geometry>
-    </visual>
-    <collision>
-      <origin xyz="0 0 -0.1" rpy="0 0 0"/>
-      <geometry>
-        <cylinder length="0.15" radius="0.045"/>
-      </geometry>
-    </collision>
-    <inertial>
-      <mass value="0.83" />
-      <origin xyz="0 0 0" />
-      <inertia ixx="0.002" ixy="0.0" ixz="0.0"
-               iyy="0.001" iyz="0.0"
-               izz="0.002" />
-    </inertial>
-  </link>
-  <xacro:rgbd_cameras topic_azure="azure" topic_kinect="kinect" parent_link="base_link"/>
+  <!-- Wheel xacro -->
+  <xacro:wheel prefix="front" suffix="left" reflect_side="1" reflect_front="1"/>
+  <xacro:wheel prefix="rear" suffix="left" reflect_side="1" reflect_front="-1"/>
+  <xacro:wheel prefix="front" suffix="right" reflect_side="-1" reflect_front="1"/>
+  <xacro:wheel prefix="rear" suffix="right" reflect_side="-1" reflect_front="-1"/>
+  <!-- add topic_kinect="kinect" for kinect camera -->
+  <xacro:rgbd_cameras topic_azure="azure" parent_link="base_link"/>
+  <xacro:imu_setup topic_imu_um7="um7/imu/data" topic_imu_azure="azure/imu/data" parent_link="base_link"/>
+  <xacro:lidar_setup topic_lidar_vlp16="vlp16/scan" topic_lidar_rplidar="rplidar/scan" parent_link="base_link"/>
   <gazebo>
     <plugin name="gazebo_ros_control" filename="libgazebo_ros_control.so">
       <robotNamespace>$(arg robot_namespace)</robotNamespace>
       <legacyModeNS>true</legacyModeNS>
-    </plugin>
-  </gazebo>
-  <gazebo>
-    <plugin name="imu_controller" filename="libhector_gazebo_ros_imu.so">
-      <robotNamespace>$(arg robot_namespace)</robotNamespace>
-      <updateRate>20.0</updateRate>
-      <bodyName>base_link</bodyName>
-      <topicName>imu/data</topicName>
-      <xyzOffset>0 0 0</xyzOffset>
-      <rpyOffset>0 0 0</rpyOffset>
-      <accelDrift>0.5 0.5 0.5</accelDrift>
-      <accelGaussianNoise>0.05 0.05 0.05</accelGaussianNoise>
-      <rateDrift>0.5 0.5 0.5 </rateDrift>
-      <rateGaussianNoise>0.05 0.05 0.05 </rateGaussianNoise>
-      <headingDrift>0.005</headingDrift>
-      <headingGaussianNoise>0.005</headingGaussianNoise>
     </plugin>
   </gazebo>
@@ -229,44 +138,3 @@
     </plugin>
   </gazebo>
-  <gazebo reference="base_scan">
-    <sensor type="ray" name="velodyne_VLP16">
-      <pose>2 0 0 0 0 0</pose>
-      <visualize>false</visualize>
-      <update_rate>10</update_rate>
-      <ray>
-        <scan>
-          <horizontal>
-            <samples>1875</samples>
-            <resolution>1</resolution>
-	    <min_angle>-${PI}</min_angle>
-	    <max_angle>${PI}</max_angle>
-          </horizontal>
-          <vertical>
-            <samples>16</samples>
-            <resolution>1</resolution>
-            <min_angle>-${15.0*PI/180.0}</min_angle>
-            <max_angle> ${15.0*PI/180.0}</max_angle>
-          </vertical>
-        </scan>
-        <range>
-          <min>0.3</min>
-          <max>2</max>
-          <resolution>0.001</resolution>
-        </range>
-        <noise>
-          <type>gaussian</type>
-          <mean>0.0</mean>
-          <stddev>0.0</stddev>
-        </noise>
-      </ray>
-      <plugin name="gazebo_ros_laser_controller" filename="libgazebo_ros_laser.so">
-	<robotNamespace>$(arg robot_namespace)</robotNamespace>
-	<topicName>scan</topicName>
-        <frameName>base_scan</frameName>
-	<min_range>0.9</min_range>
-	<max_range>2</max_range>
-        <gaussianNoise>0.008</gaussianNoise>
-      </plugin>
-    </sensor>
-  </gazebo>
 </robot>

Commit message: minor changes

File: icerobot/icerobot_description/urdf/azure_camera.urdf.xacro (robot description, xacro)
@@ -31,5 +31,5 @@
     </link>
     <joint name="azure_camera_visor_joint" type="fixed">
-      <origin xyz="0.07 0 0.025" rpy="${-PI/2-0.1} 0 ${-PI/2}"/>
+      <origin xyz="0.07 0 0.025" rpy="0 0 0"/>
       <parent link="azure_camera_body"/>
       <child link="azure_camera_visor"/>
@@ -43,5 +43,4 @@
     </joint>
     <link name="azure_imu_link"/>
- -->
     <joint name="azure_lens_gazebo_joint" type="fixed">
 	    <origin xyz="0 0 0" rpy="0 0 0"/>
@@ -49,4 +48,5 @@
       <child link="azure_camera"/>
     </joint>
+ -->
     <!-- Kinect camera joints
     <joint name="kinect_camera_joint" type="fixed">
@@ -84,18 +84,17 @@
     <xacro:macro name="depth_cam_init" params="
                frame:=cam_name           topic:=cam_topic
-               h_fov:=1.3090             v_fov:=1.1345
+               h_fov:=1.3090             v_fov:=1.2345
                min_range:=0.5            max_range:=3.86
                width:=640                height:=576
                update_rate:=30
                robot_namespace:=/">
-      <link name="${frame}" />
       <link name="${frame}_gazebo" />
       <joint name="${frame}_gazebo_joint" type="fixed">
-        <parent link="${frame}"/>
+        <parent link="${frame}_visor"/>
         <child link="${frame}_gazebo"/>
-        <origin xyz="0.0 0 0" rpy="-1.5707963267948966 0 -1.5707963267948966"/>
+	<origin xyz="0.0 0 0" rpy="${-PI/2} 0 ${-PI/2}"/>
       </joint>
-      <gazebo reference="${frame}">
-        <sensor type="depth" name="${frame}">
+      <gazebo reference="${frame}_visor">
+        <sensor type="depth" name="${frame}_gazebo">
           <update_rate>${update_rate}</update_rate>
           <camera>

File: icerobot/icerobot_gazebo/urdf/orchard_geometry.urdf.xacro (robot description, xacro)
@@ -10,5 +10,5 @@
       <origin xyz="0 0 0" rpy="0 0 0"/>
       <geometry>
-        <mesh filename="package://icerobot_gazebo/meshes/Orchard_1.dae"/>
+        <mesh filename="package://icerobot_gazebo/meshes/Orchard_2.dae"/>
       </geometry>
     </visual>
@@ -16,5 +16,5 @@
       <origin xyz="0 0 0" rpy="0 0 0"/>
       <geometry>
-        <mesh filename="package://icerobot_gazebo/meshes/Orchard_1.dae"/>
+        <mesh filename="package://icerobot_gazebo/meshes/Orchard_2.dae"/>
       </geometry>
       <surface>
